Commit message: added gazebo definitions and moveit configuration

File: robotiq_85_description/urdf/robotiq_85_gripper.urdf.xacro (robot description, xacro)
@@ -1,24 +1,21 @@
 <?xml version="1.0"?>
-<robot xmlns:xacro="http://ros.org/wiki/xacro">
+<robot name="robotiq_85_gripper" xmlns:xacro="http://ros.org/wiki/xacro">
+    <xacro:include filename="$(find robotiq_85_description)/urdf/robotiq_85_gripper.transmission.xacro" />
     <property name="pi" value="3.14159"/>
-    <xacro:macro name="robotiq_85_gripper" params="prefix">
-        <link name="${prefix}robotiq_85_root"/>
-        <!--  /\  -->
+    <xacro:macro name="robotiq_85_gripper" params="prefix parent *origin">
         <joint name="${prefix}robotiq_85_base_joint" type="fixed">
-            <parent link="${prefix}robotiq_85_root"/>
+            <parent link="${parent}"/>
             <child link="${prefix}robotiq_85_base_link"/>
-            <axis xyz="0 0 1"/>
-            <origin rpy="0.0 0.0 0.0" xyz="0.0 0.0 0.0"/>
-        </joint>
-        <!--  \/  -->
+            <xacro:insert_block name="origin"/>
+        </joint>
         <link name="${prefix}robotiq_85_base_link">
             <visual>
                 <geometry>
-                    <mesh filename="package://robotiq_85_description/meshes/robotiq_85_gripper/visual/robotiq_85_base_link.dae"/>
-                </geometry>
-            </visual>
-            <collision>
-                <geometry>
-                    <mesh filename="package://robotiq_85_description/meshes/robotiq_85_gripper/collision/robotiq_85_base_link.stl"/>
+                    <mesh filename="package://robotiq_85_description/meshes/visual/robotiq_85_base_link.dae"/>
+                </geometry>
+            </visual>
+            <collision>
+                <geometry>
+                    <mesh filename="package://robotiq_85_description/meshes/collision/robotiq_85_base_link.stl"/>
                 </geometry>
             </collision>
@@ -31,6 +28,4 @@
             </inertial>
         </link>
-        <!--  /\  -->
-        <!--  /\  -->
         <joint name="${prefix}robotiq_85_left_knuckle_joint" type="revolute">
             <parent link="${prefix}robotiq_85_base_link"/>
@@ -40,23 +35,21 @@
             <limit lower="0.0" upper="0.804" velocity="2.0" effort="1000"/>
         </joint>
-        <joint name="${prefix}robotiq_85_right_knuckle_joint" type="revolute">
+        <joint name="${prefix}robotiq_85_right_knuckle_joint" type="continuous">
             <parent link="${prefix}robotiq_85_base_link"/>
             <child link="${prefix}robotiq_85_right_knuckle_link"/>
             <axis xyz="0 0 1"/>
             <origin rpy="0.0 0.0 0.0" xyz="0.05490451627 -0.03060114443 0.0"/>
-            <limit lower="-0.804" upper="0.0" velocity="2.0" effort="1000"/>
-            <mimic joint="${prefix}robotiq_85_left_knuckle_joint" multiplier="1"/>
-        </joint>
-        <!--  \/  -->
-        <!--  \/  -->
+            <limit lower="-3.14" upper="3.14" velocity="100.0" effort="1000"/>
+            <mimic joint="${prefix}robotiq_85_left_knuckle_joint"/>
+        </joint>
         <link name="${prefix}robotiq_85_left_knuckle_link">
             <visual>
                 <geometry>
-                    <mesh filename="package://robotiq_85_description/meshes/robotiq_85_gripper/visual/robotiq_85_knuckle_link.dae"/>
-                </geometry>
-            </visual>
-            <collision>
-                <geometry>
-                    <mesh filename="package://robotiq_85_description/meshes/robotiq_85_gripper/collision/robotiq_85_knuckle_link.stl"/>
+                    <mesh filename="package://robotiq_85_description/meshes/visual/robotiq_85_knuckle_link.dae"/>
+                </geometry>
+            </visual>
+            <collision>
+                <geometry>
+                    <mesh filename="package://robotiq_85_description/meshes/collision/robotiq_85_knuckle_link.stl"/>
                 </geometry>
             </collision>
@@ -72,10 +65,10 @@
             <visual>
                 <geometry>
-                    <mesh filename="package://robotiq_85_description/meshes/robotiq_85_gripper/visual/robotiq_85_knuckle_link.dae"/>
-                </geometry>
-            </visual>
-            <collision>
-                <geometry>
-                    <mesh filename="package://robotiq_85_description/meshes/robotiq_85_gripper/collision/robotiq_85_knuckle_link.stl"/>
+                    <mesh filename="package://robotiq_85_description/meshes/visual/robotiq_85_knuckle_link.dae"/>
+                </geometry>
+            </visual>
+            <collision>
+                <geometry>
+                    <mesh filename="package://robotiq_85_description/meshes/collision/robotiq_85_knuckle_link.stl"/>
                 </geometry>
             </collision>
@@ -88,31 +81,23 @@
             </inertial>
         </link>
-        <!--  /\  -->
-        <!--  /\  -->
         <joint name="${prefix}robotiq_85_left_finger_joint" type="fixed">
             <parent link="${prefix}robotiq_85_left_knuckle_link"/>
             <child link="${prefix}robotiq_85_left_finger_link"/>
-            <axis xyz="0 0 1"/>
             <origin xyz="-0.00408552455 -0.03148604435 0.0" rpy="0 0 0" />
-            <limit lower="0" upper="2.617994" velocity="2.0" effort="1000"/>
         </joint>
         <joint name="${prefix}robotiq_85_right_finger_joint" type="fixed">
             <parent link="${prefix}robotiq_85_right_knuckle_link"/>
             <child link="${prefix}robotiq_85_right_finger_link"/>
-            <axis xyz="0 0 1"/>
             <origin xyz="-0.00408552455 -0.03148604435 0.0" rpy="0 0 0" />
-            <limit lower="0" upper="2.617994" velocity="2.0" effort="0"/>
-        </joint>
-        <!--  \/  -->
-        <!--  \/  -->
+        </joint>
         <link name="${prefix}robotiq_85_left_finger_link">
             <visual>
                 <geometry>
-                    <mesh filename="package://robotiq_85_description/meshes/robotiq_85_gripper/visual/robotiq_85_finger_link.dae"/>
-                </geometry>
-            </visual>
-            <collision>
-                <geometry>
-                    <mesh filename="package://robotiq_85_description/meshes/robotiq_85_gripper/collision/robotiq_85_finger_link.stl"/>
+                    <mesh filename="package://robotiq_85_description/meshes/visual/robotiq_85_finger_link.dae"/>
+                </geometry>
+            </visual>
+            <collision>
+                <geometry>
+                    <mesh filename="package://robotiq_85_description/meshes/collision/robotiq_85_finger_link.stl"/>
                 </geometry>
             </collision>
@@ -128,10 +113,10 @@
             <visual>
                 <geometry>
-                    <mesh filename="package://robotiq_85_description/meshes/robotiq_85_gripper/visual/robotiq_85_finger_link.dae"/>
-                </geometry>
-            </visual>
-            <collision>
-                <geometry>
-                    <mesh filename="package://robotiq_85_description/meshes/robotiq_85_gripper/collision/robotiq_85_finger_link.stl"/>
+                    <mesh filename="package://robotiq_85_description/meshes/visual/robotiq_85_finger_link.dae"/>
+                </geometry>
+            </visual>
+            <collision>
+                <geometry>
+                    <mesh filename="package://robotiq_85_description/meshes/collision/robotiq_85_finger_link.stl"/>
                 </geometry>
             </collision>
@@ -144,33 +129,29 @@
             </inertial>
         </link>
-        <!--  /\  -->
-        <!--  /\  -->
-        <joint name="${prefix}robotiq_85_left_inner_knuckle_joint" type="revolute">
+        <joint name="${prefix}robotiq_85_left_inner_knuckle_joint" type="continuous">
             <parent link="${prefix}robotiq_85_base_link"/>
             <child link="${prefix}robotiq_85_left_inner_knuckle_link"/>
             <axis xyz="0 0 1"/>
             <origin xyz="0.06142 0.0127 0" rpy="${pi} 0.0 0.0" />
-            <limit lower="-0.804" upper="0.0" velocity="2.0" effort="1000"/>
+            <limit lower="-3.14" upper="3.14" velocity="100.0" effort="0.1"/>
             <mimic joint="${prefix}robotiq_85_left_knuckle_joint" offset="0"/>
         </joint>
-        <joint name="${prefix}robotiq_85_right_inner_knuckle_joint" type="revolute">
+        <joint name="${prefix}robotiq_85_right_inner_knuckle_joint" type="continuous">
             <parent link="${prefix}robotiq_85_base_link"/>
             <child link="${prefix}robotiq_85_right_inner_knuckle_link"/>
             <axis xyz="0 0 1"/>
             <origin xyz="0.06142 -0.0127 0" rpy="0 0 0"/>
-            <limit lower="0" upper="0.804" velocity="2.0" effort="1000"/>
+            <limit lower="-3.14" upper="3.14" velocity="100.0" effort="0.1"/>
             <mimic joint="${prefix}robotiq_85_left_knuckle_joint" offset="0"/>
         </joint>
-        <!--  \/  -->
-        <!--  \/  -->
         <link name="${prefix}robotiq_85_left_inner_knuckle_link">
             <visual>
                 <geometry>
-                    <mesh filename="package://robotiq_85_description/meshes/robotiq_85_gripper/visual/robotiq_85_inner_knuckle_link.dae"/>
-                </geometry>
-            </visual>
-            <collision>
-                <geometry>
-                    <mesh filename="package://robotiq_85_description/meshes/robotiq_85_gripper/collision/robotiq_85_inner_knuckle_link.stl"/>
+                    <mesh filename="package://robotiq_85_description/meshes/visual/robotiq_85_inner_knuckle_link.dae"/>
+                </geometry>
+            </visual>
+            <collision>
+                <geometry>
+                    <mesh filename="package://robotiq_85_description/meshes/collision/robotiq_85_inner_knuckle_link.stl"/>
                 </geometry>
             </collision>
@@ -186,10 +167,10 @@
             <visual>
                 <geometry>
-                    <mesh filename="package://robotiq_85_description/meshes/robotiq_85_gripper/visual/robotiq_85_inner_knuckle_link.dae"/>
-                </geometry>
-            </visual>
-            <collision>
-                <geometry>
-                    <mesh filename="package://robotiq_85_description/meshes/robotiq_85_gripper/collision/robotiq_85_inner_knuckle_link.stl"/>
+                    <mesh filename="package://robotiq_85_description/meshes/visual/robotiq_85_inner_knuckle_link.dae"/>
+                </geometry>
+            </visual>
+            <collision>
+                <geometry>
+                    <mesh filename="package://robotiq_85_description/meshes/collision/robotiq_85_inner_knuckle_link.stl"/>
                 </geometry>
             </collision>
@@ -202,33 +183,29 @@
             </inertial>
         </link>
-        <!--  /\  -->
-        <!--  /\  -->
-        <joint name="${prefix}robotiq_85_left_finger_tip_joint" type="revolute">
+        <joint name="${prefix}robotiq_85_left_finger_tip_joint" type="continuous">
             <parent link="${prefix}robotiq_85_left_inner_knuckle_link"/>
             <child link="${prefix}robotiq_85_left_finger_tip_link"/>
             <axis xyz="0 0 1"/>
             <origin xyz="0.04303959807 -0.03759940821 0.0" rpy="0.0 0.0 0.0"/>
-            <limit lower="0" upper="1.5707" velocity="2.0" effort="1000"/>
+            <limit lower="-3.14" upper="3.14" velocity="100.0" effort="0.1"/>
             <mimic joint="${prefix}robotiq_85_left_knuckle_joint" multiplier="-1"/>
         </joint>
-        <joint name="${prefix}robotiq_85_right_finger_tip_joint" type="revolute">
+        <joint name="${prefix}robotiq_85_right_finger_tip_joint" type="continuous">
             <parent link="${prefix}robotiq_85_right_inner_knuckle_link"/>
             <child link="${prefix}robotiq_85_right_finger_tip_link"/>
             <axis xyz="0 0 1"/>
             <origin rpy="0.0 0.0 0.0" xyz="0.04303959807 -0.03759940821  0.0"/>
-            <limit lower="0" upper="1.5707" velocity="2.0" effort="1000"/>
+            <limit lower="-3.14" upper="3.14" velocity="100.0" effort="0.1"/>
             <mimic joint="${prefix}robotiq_85_left_knuckle_joint" multiplier="-1"/>
         </joint>
-        <!--  \/  -->
-        <!--  \/  -->
         <link name="${prefix}robotiq_85_left_finger_tip_link">
             <visual>
                 <geometry>
-                    <mesh filename="package://robotiq_85_description/meshes/robotiq_85_gripper/visual/robotiq_85_finger_tip_link.dae"/>
-                </geometry>
-            </visual>
-            <collision>
-                <geometry>
-                    <mesh filename="package://robotiq_85_description/meshes/robotiq_85_gripper/collision/robotiq_85_finger_tip_link.stl"/>
+                    <mesh filename="package://robotiq_85_description/meshes/visual/robotiq_85_finger_tip_link.dae"/>
+                </geometry>
+            </visual>
+            <collision>
+                <geometry>
+                    <mesh filename="package://robotiq_85_description/meshes/collision/robotiq_85_finger_tip_link.stl"/>
                 </geometry>
             </collision>
@@ -244,10 +221,10 @@
             <visual>
                 <geometry>
-                    <mesh filename="package://robotiq_85_description/meshes/robotiq_85_gripper/visual/robotiq_85_finger_tip_link.dae"/>
-                </geometry>
-            </visual>
-            <collision>
-                <geometry>
-                    <mesh filename="package://robotiq_85_description/meshes/robotiq_85_gripper/collision/robotiq_85_finger_tip_link.stl"/>
+                    <mesh filename="package://robotiq_85_description/meshes/visual/robotiq_85_finger_tip_link.dae"/>
+                </geometry>
+            </visual>
+            <collision>
+                <geometry>
+                    <mesh filename="package://robotiq_85_description/meshes/collision/robotiq_85_finger_tip_link.stl"/>
                 </geometry>
             </collision>
@@ -260,4 +237,5 @@
             </inertial>
         </link>
+        <xacro:robotiq_85_gripper_transmission prefix="${prefix}" />
     </xacro:macro>
 </robot>

File: robotiq_85_description/urdf/robotiq_85_gripper.xacro (robot description, xacro)
@@ -2,4 +2,38 @@
 <robot name="robotiq_85_gripper" xmlns:xacro="http://ros.org/wiki/xacro">
     <xacro:include filename="$(find robotiq_85_description)/urdf/robotiq_85_gripper.urdf.xacro" />
-    <xacro:robotiq_85_gripper prefix=""/>
+    <gazebo>
+        <plugin name="gazebo_ros_control" filename="libgazebo_ros_control.so">
+            <robotNamespace>/</robotNamespace>
+        </plugin>
+    </gazebo>
+    <link name="world"/>
+    <joint name="world_fixed" type="fixed">
+        <origin xyz="0 0 0" rpy="0 0 0"/>
+        <parent link="world"/>
+        <child link="gripper_root_link"/>
+    </joint>
+    <link name="gripper_root_link">
+        <visual>
+            <origin xyz="0 0 0.5" rpy="0 0 0"/>
+            <geometry>
+                <box size="0.1 0.1 1.0"/>
+            </geometry>
+        </visual>
+        <collision>
+            <origin xyz="0 0 0.5" rpy="0 0 0"/>
+            <geometry>
+                <box size="0.1 0.1 1.0"/>
+            </geometry>
+        </collision>
+        <inertial>
+            <mass value="1e2" />
+            <origin xyz="0.0 0.0 0.0" />
+            <inertia ixx = "0.000001" ixy = "0.000000" ixz = "0.000000"
+                     iyx = "0.000000" iyy = "0.000001" iyz = "0.000000"
+                     izx = "0.000000" izy = "0.000000" izz = "0.000001" />
+        </inertial>
+    </link>
+    <xacro:robotiq_85_gripper prefix="" parent="gripper_root_link" >
+        <origin xyz="0.05 0 0.85" rpy="0 0 0"/>
+    </xacro:robotiq_85_gripper>
 </robot>
